Commit message: change lidar param to URG-04LX-UG01

File: robots/vmegarover.urdf.xacro (robot description, xacro)
@@ -1,7 +1,7 @@
 <?xml version="1.0"?>
 <robot name="vmegarover" xmlns:xacro="http://ros.org/wiki/xacro">
-  <xacro:include filename="$(find megarover_samples)/urdf/body/vbody.urdf.xacro"/>
-  <xacro:include filename="$(find megarover_samples)/urdf/wheel/vwheel.urdf.xacro"/>
-  <xacro:include filename="$(find megarover_samples)/urdf/lrf/lrf.urdf.xacro"/>
+  <xacro:include filename="$(find kaitlv)/urdf/body/vbody.urdf.xacro"/>
+  <xacro:include filename="$(find kaitlv)/urdf/wheel/vwheel.urdf.xacro"/>
+  <xacro:include filename="$(find kaitlv)/urdf/lrf/lrf.urdf.xacro"/>
   <!-- =============== Link & Joint =============== -->
   <!-- Base -->
@@ -23,5 +23,5 @@
   <!-- Front LRF -->
   <xacro:lrf_v0 prefix="front" parent="base_link">
-    <origin xyz="0.099 0 0.1015"/>
+    <origin xyz="0.099 0 0.1815"/>
   </xacro:lrf_v0>
   <!-- Front LRF Upper-->
@@ -55,5 +55,5 @@
   <!-- LRF -->
   <xacro:lrf_gazebo_v0 prefix="front"
-                       min_rad="-1.57" max_rad="1.57"
+                       min_rad="-2.09" max_rad="2.09"
                        min_range="0.06" max_range="4.0"/>
   <!-- xacro:lrf_gazebo_v0 prefix="rear"

File: urdf/lrf/lrf.gazebo.xacro (robot description, xacro)
@@ -10,5 +10,5 @@
           <scan>
             <horizontal>
-              <samples>1000</samples>
+              <samples>682</samples>
               <resolution>1</resolution>
               <min_angle>${min_rad}</min_angle>

File: urdf/lrf/lrf.urdf.xacro (robot description, xacro)
@@ -1,6 +1,6 @@
 <?xml version="1.0"?>
 <robot xmlns:xacro="http://ros.org/wiki/xacro">
-  <xacro:include filename="$(find megarover_samples)/urdf/common.xacro"/>
-  <xacro:include filename="$(find megarover_samples)/urdf/lrf/lrf.gazebo.xacro"/>
+  <xacro:include filename="$(find kaitlv)/urdf/common.xacro"/>
+  <xacro:include filename="$(find kaitlv)/urdf/lrf/lrf.gazebo.xacro"/>
   <xacro:macro name="lrf_v0" params="prefix parent *joint_origin">
     <joint name="${prefix}_lrf_joint" type="fixed">
@@ -12,10 +12,10 @@
       <visual>
         <geometry>
-          <mesh filename="package://megarover_samples/meshes/dae/lrf.dae"/>
+          <mesh filename="package://kaitlv/meshes/dae/lrf.dae"/>
         </geometry>
       </visual>
       <collision>
         <geometry>
-          <mesh filename="package://megarover_samples/meshes/stl/lrf.stl"/>
+          <mesh filename="package://kaitlv/meshes/stl/lrf.stl"/>
         </geometry>
       </collision>
